File: pcb/keyboard_pcb.kicad_sch (KiCad schematic)
At the start: 23 parts, among them J1 TRRS, K00 KEYSW, K01 KEYSW, K02 KEYSW, K03 KEYSW, K04 KEYSW, K05 KEYSW, K10 KEYSW, K11 KEYSW, K12 KEYSW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

Commit message: RP2040 symbol& footprint eingebaut
Parts:
- added U?: WeAct-RP2040-Pico, WeAct-RP2040-Pico:WeAct-RP2040-Pico, symbol WeAct-RP2040_prj:WeAct-RP2040-Pico
Changed lines of the file:
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@@
     (pin "4")
+  )
+  (symbol (lib_id "WeAct-RP2040_prj:WeAct-RP2040-Pico") (at 110.49 106.68 0) (unit 1)
+    (in_bom yes) (on_board yes) (fields_autoplaced)
+    (property "Reference" "U?" (id 0) (at 110.49 82.7872 0))
+    (property "Value" "WeAct-RP2040-Pico" (id 1) (at 110.49 85.3241 0))
+    (property "Footprint" "WeAct-RP2040-Pico:WeAct-RP2040-Pico" (id 2) (at 110.49 106.68 0)
+      (effects (font (size 1.27 1.27)) hide)
+    )
+    (property "Datasheet" "https://github.com/WeActStudio/WeActStudio.RP2040CoreBoard/tree/master" (id 3) (at 110.49 106.68 0)
+      (effects (font (size 1.27 1.27)) hide)
+    )
+    (pin "1")
+    (pin "10")
+    (pin "11")
+    (pin "12")
+    (pin "13")
+    (pin "14")
+    (pin "15")
+    (pin "16")
+    (pin "17")
+    (pin "18")
+    (pin "19")
+    (pin "2")
+    (pin "20")
+    (pin "21")
+    (pin "22")
+    (pin "23")
+    (pin "24")
+    (pin "25")
+    (pin "26")
+    (pin "27")
+    (pin "28")
+    (pin "29")
+    (pin "3")
+    (pin "30")
+    (pin "31")
+    (pin "32")
+    (pin "33")
+    (pin "34")
+    (pin "35")
+    (pin "36")
+    (pin "37")
+    (pin "38")
+    (pin "39")
+    (pin "4")
+    (pin "40")
+    (pin "41")
+    (pin "42")
+    (pin "43")
+    (pin "44")
+    (pin "5")
+    (pin "6")
+    (pin "7")
+    (pin "8")
+    (pin "9")
   )
   (symbol (lib_id "keyboard_parts:KEYSW") (at 137.16 60.96 0) (mirror y) (unit 1)
@@
       (reference "U1") (unit 1) (value "YAAJ_WeAct_BlackPill_Part_Like") (footprint "Footprints:YAAJ_WeAct_BlackPill_2")
     )
-  )
+    (path "/90ca3f28-9cc2-4ba4-a917-c792fc534948"
+      (reference "U?") (unit 1) (value "WeAct-RP2040-Pico") (footprint "WeAct-RP2040-Pico:WeAct-RP2040-Pico")
+    )
+  )

Commit message: WIP: adding  RP2040 + oled
Parts:
- added J2: Conn_01x04_Female, symbol Connector:Conn_01x04_Female
- U2: renamed from U?; footprint WeAct-RP2040-Pico:WeAct-RP2040-Pico -> rp2040:WeAct-RP2040-Pico
- renumbered K00 to K0, K01 to K1, K02 to K2, K03 to K3, K04 to K4, K05 to K5
Connections:
- net +3V3: now also U2.37 (3V3), J2.2 (Pin_2); no longer U1.20 (3V3), U1.38 (3V3)
- net GND: now also U2.13 (GND), U2.18 (GND), U2.23 (GND), U2.28 (GND), U2.33 (GND), U2.38 (GND), U2.41 (GND), U2.8 (GND), J2.1 (Pin_1); no longer U1.19 (GND), U1.39 (GND)
- net RX: now also U2.17 (GP13); no longer U1.15 (PB7)
- net TX: now also U2.16 (GP12); no longer U1.14 (PB6)
- net k00: no longer U1.35 (PB1)
- net k01: no longer U1.37 (PB10)
- net k02: no longer U1.5 (PA8)
- net k03: no longer U1.4 (PB15)
- net k04: no longer U1.3 (PB14)
- net k05: no longer U1.2 (PB13)
- net k10: no longer U1.17 (PB9)
- net k11: no longer U1.16 (PB8)
- net k12: no longer U1.13 (PB5)
- net k13: no longer U1.12 (PB4)
- net k14: no longer U1.11 (PB3)
- net k15: no longer U1.10 (PA15)
- net k20: no longer U1.29 (PA3)
- net k21: no longer U1.30 (PA4)
- net k22: no longer U1.31 (PA5)
- net k23: no longer U1.32 (PA6)
- net k24: no longer U1.33 (PA7)
- net k25: no longer U1.34 (PB0)
- net k30: no longer U1.28 (PA2)
- net k31: no longer U1.27 (PA1)
- net k32: no longer U1.26 (PA0)
- net SDA: now reaches U2.19 (GP14)
- net SDA: now also J2.4 (Pin_4)
- net SCK: now reaches U2.20 (GP15)
- net SCK: now also J2.3 (Pin_3)
Other:
- moved on the sheet: U2

Commit message: WIP: adding  RP2040 + oled
Parts:
- J2: footprint (none) -> Connector_PinSocket_2.54mm:PinSocket_1x04_P2.54mm_Vertical
Changed lines of the file:
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@@
     (property "Reference" "J2" (id 0) (at 47.625 136.813 0))
     (property "Value" "Conn_01x04_Female" (id 1) (at 47.625 139.3499 0))
-    (property "Footprint" "" (id 2) (at 46.99 146.05 0)
+    (property "Footprint" "Connector_PinSocket_2.54mm:PinSocket_1x04_P2.54mm_Vertical" (id 2) (at 46.99 146.05 0)
       (effects (font (size 1.27 1.27)) hide)
     )
@@
     )
     (path "/43fed586-9749-4fb0-91ff-a0b521d57cd5"
-      (reference "J2") (unit 1) (value "Conn_01x04_Female") (footprint "")
+      (reference "J2") (unit 1) (value "Conn_01x04_Female") (footprint "Connector_PinSocket_2.54mm:PinSocket_1x04_P2.54mm_Vertical")
     )
     (path "/2cd2ee6e-af2a-43ce-aa7e-58b5c17fc3c8"
